Commit message: split the model and semantics into macros for robots built on the LeKiwi
The ground and the LeKiwi's semantic description (groups, poses, end
effectors, disabled collision pairs) are now xacro macros in
config/ground.xacro and config/lekiwi_semantic.xacro; config/lekiwi.srdf
becomes config/lekiwi.srdf.xacro, which instantiates the macro. A robot that
adds parts to the LeKiwi can include both and add only the collision pairs
of its own links, instead of copying the SRDF and keeping it in sync.

lekiwi_moveit_config() in launch/moveit_config.py takes the package, robot
name, URDF and SRDF, so such a robot's MoveIt launches reuse it with its own
files. The defaults give the stock LeKiwi config as before.

scripts/compute_disabled_collisions.py, installed with the package, is the
tool used to generate the disabled collision pairs: it samples the robot's
poses with moveit_py, and with --new-only prints only pairs the SRDF does not
have yet, which is what an extension needs after adding links.

File: config/lekiwi.urdf.xacro (robot description, xacro)
@@ -5,29 +5,5 @@
        keep using lekiwi_bringup/urdf/lekiwi.urdf.xacro, and the joints are the same. -->
   <xacro:include filename="$(find lekiwi_bringup)/urdf/lekiwi.urdf.xacro"/>
-  <!-- Ground: base_footprint is at floor level, so the floor moves with the robot as it drives.
-       The top surface is at z = 0. -->
-  <xacro:property name="ground_size" value="2.0"/>
-  <xacro:property name="ground_thickness" value="0.01"/>
-  <link name="ground">
-    <visual>
-      <origin xyz="0 0 ${-ground_thickness/2}" rpy="0 0 0"/>
-      <geometry>
-        <box size="${ground_size} ${ground_size} ${ground_thickness}"/>
-      </geometry>
-      <material name="lekiwi_moveit_ground">
-        <color rgba="0.35 0.35 0.35 0.4"/>
-      </material>
-    </visual>
-    <collision>
-      <origin xyz="0 0 ${-ground_thickness/2}" rpy="0 0 0"/>
-      <geometry>
-        <box size="${ground_size} ${ground_size} ${ground_thickness}"/>
-      </geometry>
-    </collision>
-  </link>
-  <joint name="ground_joint" type="fixed">
-    <parent link="base_footprint"/>
-    <child link="ground"/>
-    <origin xyz="0 0 0" rpy="0 0 0"/>
-  </joint>
+  <xacro:include filename="$(find lekiwi_moveit_config)/config/ground.xacro"/>
+  <xacro:lekiwi_ground/>
 </robot>
